Commit message: Update urdf

File: src/puzzlebot_description/urdf/puzzlebot_mcr2.urdf.xacro (robot description, xacro)
@@ -130,11 +130,4 @@
     </inertial>
   </link>
-  <!-- IMU link -->
-  <link name="imu_link">
-    <inertial>
-      <mass value="0.01"/>
-      <inertia ixx="1e-7" ixy="0" ixz="0" iyy="1e-7" iyz="0" izz="1e-7"/>
-    </inertial>
-  </link>
   <!-- ==================== JOINTS ==================== -->
   <!-- base_footprint -> base_link -->
@@ -176,10 +169,4 @@
     <origin xyz="0.112 0 0.065" rpy="0 0 0"/>
   </joint>
-  <!-- base_link -> imu_link -->
-  <joint name="imu_joint" type="fixed">
-    <parent link="base_link"/>
-    <child link="imu_link"/>
-    <origin xyz="0.0 0.0 0.04" rpy="0.0 0.0 0.0"/>
-  </joint>
   <!-- Materials -->
   <material name="dark_grey">
