Commit message: Add warehouse model and lifter mechanism to puzzlebot_description

File: src/puzzlebot_description/urdf/puzzlebot_ros2_control.xacro (robot description, xacro)
@@ -15,4 +15,21 @@
       </xacro:unless>
     </xacro:if>
+    <!-- Lifter prismatic joints -->
+    <joint name="mast_inner_joint">
+      <command_interface name="effort">
+        <param name="min">-100.0</param>
+        <param name="max">100.0</param>
+      </command_interface>
+      <state_interface name="position"/>
+      <state_interface name="velocity"/>
+    </joint>
+    <joint name="carriage_joint">
+      <command_interface name="effort">
+        <param name="min">-50.0</param>
+        <param name="max">50.0</param>
+      </command_interface>
+      <state_interface name="position"/>
+      <state_interface name="velocity"/>
+    </joint>
     <!-- Wheel joints -->
     <joint name="wheel_left_joint">
