Commit message: Updated meshes

File: src/puzzlebot_description/urdf/lifter.urdf.xacro (robot description, xacro)
@@ -15,12 +15,11 @@
   <link name="world"/>
   <!-- Outer mast / fork base (4-mast-1.stl) ─ fixed reference
-       STL lies flat (long axis in mesh-Y=170mm).  rpy="1.5708 0 0" rotates
-       mesh-Y → world-Z so the mast stands upright (170mm tall).
-       xyz centres the mesh on the link origin (computed from bounding box). -->
+       rpy="1.5708 3.14159 0" = Rx(90°) then Ry(180°): stands upright and
+       flipped 180° on Y. xyz re-centred for the flipped orientation. -->
   <link name="lifter_base_link">
     <visual>
-      <origin xyz="-0.1125 0.0112 -0.1125" rpy="1.5708 0 0"/>
+      <origin xyz="-0.1125 -0.0112 0.1125" rpy="1.5708 3.14159 3.14159"/>
       <geometry>
-        <mesh filename="package://puzzlebot_description/meshes/4-mast-1.stl"
+        <mesh filename="package://puzzlebot_description/meshes/lifter/outer_mast.stl"
               scale="${s} ${s} ${s}"/>
       </geometry>
@@ -35,12 +34,12 @@
     </inertial>
   </link>
-  <!-- Inner mast (7-mast-2.stl) ─ slides vertically inside outer mast
-       Same rotation: long axis (155mm) becomes Z.  Narrower than outer mast
-       so it nests cleanly inside (49mm < 55mm wide, 11.6mm < 22.4mm deep). -->
+  <!-- Inner mast (Frantic Albar-Hillar (9).stl) ─ slides vertically inside outer mast
+       Long axis (171mm) in mesh-Y → world-Z via rpy="1.5708 0 0".
+       xyz centres the mesh on the link origin (bounding box: X:41-90, Y:-65.5..105.5, Z:0-11.6). -->
   <link name="mast_inner_link">
     <visual>
-      <origin xyz="-0.1125 0.0058 -0.1125" rpy="1.5708 0 0"/>
+      <origin xyz="-0.0655 0.0058 -0.0050" rpy="1.5708 0 0"/>
       <geometry>
-        <mesh filename="package://puzzlebot_description/meshes/7-mast-2.stl"
+        <mesh filename="package://puzzlebot_description/meshes/lifter/mast_inner.stl"
               scale="${s} ${s} ${s}"/>
       </geometry>
@@ -63,5 +62,5 @@
       <origin xyz="-0.1125 -0.11343 -0.02793" rpy="0 0 0"/>
       <geometry>
-        <mesh filename="package://puzzlebot_description/meshes/8-carriage.stl"
+        <mesh filename="package://puzzlebot_description/meshes/lifter/carriage.stl"
               scale="${s} ${s} ${s}"/>
       </geometry>
@@ -74,4 +73,40 @@
       <inertia ixx="0.001" ixy="0" ixz="0"
                iyy="0.001" iyz="0" izz="0.001"/>
+    </inertial>
+  </link>
+  <!-- Camera pan holder (camera_holder.stl) — upright bracket, rotates on mast
+       Bottom of bracket (mesh-Y=59mm) sits at z=0 (= inner mast top / joint origin).
+       Top at z=0.0225m. Camera mounts above. -->
+  <link name="cam_holder_link">
+    <visual>
+      <origin xyz="0.0285 -0.0055 0.0715" rpy="-1.5708 0 0"/>
+      <geometry>
+        <mesh filename="package://puzzlebot_description/meshes/lifter/camera_holder.stl"
+              scale="${s} ${s} ${s}"/>
+      </geometry>
+      <material name="light_grey">
+        <color rgba="0.80 0.80 0.75 1.0"/>
+      </material>
+    </visual>
+    <inertial>
+      <mass value="0.01"/>
+      <inertia ixx="1e-6" ixy="0" ixz="0" iyy="1e-6" iyz="0" izz="1e-6"/>
+    </inertial>
+  </link>
+  <!-- Mast camera (camera.stl) — fixed to pan holder, rotates with it -->
+  <link name="mast_camera_link">
+    <visual>
+      <origin xyz="-0.0005 0.0290 0.0005" rpy="-1.5708 0 3.14159"/>
+      <geometry>
+        <mesh filename="package://puzzlebot_description/meshes/lifter/camera.stl"
+              scale="${s} ${s} ${s}"/>
+      </geometry>
+      <material name="black">
+        <color rgba="0.1 0.1 0.1 1.0"/>
+      </material>
+    </visual>
+    <inertial>
+      <mass value="0.01"/>
+      <inertia ixx="1e-6" ixy="0" ixz="0" iyy="1e-6" iyz="0" izz="1e-6"/>
     </inertial>
   </link>
@@ -107,4 +142,17 @@
     <limit lower="0.0" upper="0.10" effort="50.0" velocity="0.10"/>
   </joint>
+  <!-- Pan holder: revolute X at top of inner mast (z=0.085 ≈ mast top at 85.5mm) -->
+  <joint name="cam_holder_joint" type="fixed">
+    <parent link="mast_inner_link"/>
+    <child  link="cam_holder_link"/>
+    <origin xyz="0 0 0.105" rpy="0.7854 0 0"/>
+  </joint>
+  <!-- Camera: fixed to pan holder, sits on top of bracket
+       z=0.030: bracket top (0.0225) + half camera height (0.007) = 0.0295 ≈ 0.030m -->
+  <joint name="mast_camera_joint" type="fixed">
+    <parent link="cam_holder_link"/>
+    <child  link="mast_camera_link"/>
+    <origin xyz="0 0 0.033" rpy="0 0 0"/>
+  </joint>
   <!-- ═══════════════════════ MATERIALS ═══════════════════════ -->
   <material name="off_white">
@@ -114,3 +162,6 @@
     <color rgba="0.80 0.80 0.75 1.0"/>
   </material>
+  <material name="black">
+    <color rgba="0.1 0.1 0.1 1.0"/>
+  </material>
 </robot>

File: src/puzzlebot_description/urdf/puzzlebot_gazebo.xacro (robot description, xacro)
@@ -103,4 +103,32 @@
     </sensor>
   </gazebo>
+  <!-- Mast camera sensor -->
+  <gazebo reference="mast_camera_link">
+    <sensor name="mast_camera" type="camera">
+      <pose>0 0 0 0 0 -1.5708</pose>
+      <always_on>true</always_on>
+      <visualize>true</visualize>
+      <update_rate>30</update_rate>
+      <topic>/mast_camera/image_raw</topic>
+      <gz_frame_id>mast_camera_link</gz_frame_id>
+      <camera>
+        <horizontal_fov>1.047</horizontal_fov>  <!-- 60 deg -->
+        <image>
+          <width>640</width>
+          <height>480</height>
+          <format>R8G8B8</format>
+        </image>
+        <clip>
+          <near>0.05</near>
+          <far>10.0</far>
+        </clip>
+        <noise>
+          <type>gaussian</type>
+          <mean>0.0</mean>
+          <stddev>0.007</stddev>
+        </noise>
+      </camera>
+    </sensor>
+  </gazebo>
   <!-- 2D Lidar sensor -->
   <gazebo reference="lidar_link">

File: src/puzzlebot_description/urdf/puzzlebot_with_lifter.urdf.xacro (robot description, xacro)
@@ -160,7 +160,7 @@
   <link name="lifter_base_link">
     <visual>
-      <origin xyz="-0.1125 0.0112 -0.1125" rpy="1.5708 0 0"/>
-      <geometry>
-        <mesh filename="package://puzzlebot_description/meshes/4-mast-1.stl"
+      <origin xyz="-0.1125 -0.0112 0.1125" rpy="1.5708 3.14159 3.14159"/>
+      <geometry>
+        <mesh filename="package://puzzlebot_description/meshes/lifter/outer_mast.stl"
               scale="${s} ${s} ${s}"/>
       </geometry>
@@ -182,11 +182,11 @@
     </inertial>
   </link>
-  <!-- Inner mast (7-mast-2.stl)
-       Physical size in world frame: 49 × 11.6 × 155.5 mm -->
+  <!-- Inner mast (Frantic Albar-Hillar (9).stl)
+       Physical size in world frame: 49 × 11.6 × 171 mm -->
   <link name="mast_inner_link">
     <visual>
-      <origin xyz="-0.1125 0.0058 -0.1125" rpy="1.5708 0 0"/>
-      <geometry>
-        <mesh filename="package://puzzlebot_description/meshes/7-mast-2.stl"
+      <origin xyz="-0.0655 0.0058 -0.0050" rpy="1.5708 0 0"/>
+      <geometry>
+        <mesh filename="package://puzzlebot_description/meshes/lifter/mast_inner.stl"
               scale="${s} ${s} ${s}"/>
       </geometry>
@@ -198,5 +198,5 @@
       <origin xyz="0 0 0" rpy="0 0 0"/>
       <geometry>
-        <box size="0.049 0.0116 0.1555"/>
+        <box size="0.049 0.0116 0.171"/>
       </geometry>
     </collision>
@@ -214,5 +214,5 @@
       <origin xyz="-0.1125 -0.11343 -0.02793" rpy="0 0 0"/>
       <geometry>
-        <mesh filename="package://puzzlebot_description/meshes/8-carriage.stl"
+        <mesh filename="package://puzzlebot_description/meshes/lifter/carriage.stl"
               scale="${s} ${s} ${s}"/>
       </geometry>
@@ -232,4 +232,52 @@
       <inertia ixx="0.0000207" ixy="0" ixz="0"
                iyy="0.0000159" iyz="0" izz="0.0000262"/>
+    </inertial>
+  </link>
+  <!-- Camera pan holder (camera_holder.stl) — rotates on top of inner mast -->
+  <link name="cam_holder_link">
+    <visual>
+      <origin xyz="0.0285 -0.0055 0.0715" rpy="-1.5708 0 0"/>
+      <geometry>
+        <mesh filename="package://puzzlebot_description/meshes/lifter/camera_holder.stl"
+              scale="${s} ${s} ${s}"/>
+      </geometry>
+      <material name="light_grey">
+        <color rgba="0.80 0.80 0.75 1.0"/>
+      </material>
+    </visual>
+    <collision>
+      <origin xyz="0 0 0.01125" rpy="0 0 0"/>
+      <geometry>
+        <box size="0.041 0.009 0.0225"/>
+      </geometry>
+    </collision>
+    <inertial>
+      <origin xyz="0 0 0.01125" rpy="0 0 0"/>
+      <mass value="0.01"/>
+      <inertia ixx="1e-6" ixy="0" ixz="0" iyy="1e-6" iyz="0" izz="1e-6"/>
+    </inertial>
+  </link>
+  <!-- Mast camera (camera.stl) — fixed to the pan holder -->
+  <link name="mast_camera_link">
+    <visual>
+      <origin xyz="-0.0005 0.0290 0.0005" rpy="-1.5708 0 3.14159"/>
+      <geometry>
+        <mesh filename="package://puzzlebot_description/meshes/lifter/camera.stl"
+              scale="${s} ${s} ${s}"/>
+      </geometry>
+      <material name="black">
+        <color rgba="0.1 0.1 0.1 1.0"/>
+      </material>
+    </visual>
+    <collision>
+      <origin xyz="0 0 0" rpy="0 0 0"/>
+      <geometry>
+        <box size="0.041 0.041 0.014"/>
+      </geometry>
+    </collision>
+    <inertial>
+      <origin xyz="0 0 0" rpy="0 0 0"/>
+      <mass value="0.01"/>
+      <inertia ixx="1e-6" ixy="0" ixz="0" iyy="1e-6" iyz="0" izz="1e-6"/>
     </inertial>
   </link>
@@ -301,4 +349,17 @@
     <dynamics damping="10.0" friction="2.0"/>
   </joint>
+  <!-- Pan holder: revolute around X at top of inner mast -->
+  <joint name="cam_holder_joint" type="fixed">
+    <parent link="mast_inner_link"/>
+    <child  link="cam_holder_link"/>
+    <origin xyz="0 0 0.105" rpy="0.7854 0 0"/>
+  </joint>
+  <!-- Camera: fixed to the pan holder, sits on top of bracket
+       z=0.030: bracket top (0.0225) + half camera height (0.007) = 0.0295 ≈ 0.030m -->
+  <joint name="mast_camera_joint" type="fixed">
+    <parent link="cam_holder_link"/>
+    <child  link="mast_camera_link"/>
+    <origin xyz="0 0 0.033" rpy="0 0 0"/>
+  </joint>
   <!-- ==================== MATERIALS ==================== -->
   <material name="dark_grey">
