Commit message: Gazebo correcto, rviz igual y simulacion de lidar bien

File: src/description/urdf/puzzlebot.urdf.xacro (robot description, xacro)
@@ -5,7 +5,7 @@
   <xacro:arg name="is_sim" default="true"/>
   <!-- Include Gazebo plugins -->
-  <xacro:include filename="$(find puzzlebot_description)/urdf/puzzlebot_gazebo.xacro" />
+  <xacro:include filename="$(find description)/urdf/puzzlebot_gazebo.xacro" />
   <!-- Include ros2_control -->
-  <xacro:include filename="$(find puzzlebot_description)/urdf/puzzlebot_ros2_control.xacro" />
+  <xacro:include filename="$(find description)/urdf/puzzlebot_ros2_control.xacro" />
   <!-- ==================== PROPERTIES ==================== -->
   <xacro:property name="wheel_radius" value="0.05"/>
@@ -47,5 +47,5 @@
     <visual>
       <geometry>
-        <mesh filename="package://puzzlebot_description/meshes/Puzzlebot_Jetson_Lidar_Edition_Base.stl"/>
+        <mesh filename="package://description/meshes/Puzzlebot_Jetson_Lidar_Edition_Base.stl"/>
       </geometry>
       <material name="dark_grey">
@@ -65,5 +65,5 @@
       <origin xyz="0 0 0" rpy="-1.5708 0 0"/>
       <geometry>
-        <mesh filename="package://puzzlebot_description/meshes/Puzzlebot_Wheel.stl"/>
+        <mesh filename="package://description/meshes/Puzzlebot_Wheel.stl"/>
       </geometry>
       <material name="grey">
@@ -84,5 +84,5 @@
       <origin xyz="0 0 0" rpy="1.5708 0 0"/>
       <geometry>
-        <mesh filename="package://puzzlebot_description/meshes/Puzzlebot_Wheel.stl"/>
+        <mesh filename="package://description/meshes/Puzzlebot_Wheel.stl"/>
       </geometry>
       <material name="grey">
@@ -98,9 +98,12 @@
   </link>
   <!-- Caster wheel -->
+  <!-- Link origin is at the bracket mount point.
+       Ball center is +0.0057m above origin (from mesh analysis),
+       ball radius is 0.0115m. Collision sphere is offset to ball center. -->
   <link name="caster_link">
-    <xacro:sphere_inertia m="${caster_mass}" r="0.015"/>
-    <visual>
-      <geometry>
-        <mesh filename="package://puzzlebot_description/meshes/Puzzlebot_Caster_Wheel.stl"/>
+    <xacro:sphere_inertia m="${caster_mass}" r="0.0115"/>
+    <visual>
+      <geometry>
+        <mesh filename="package://description/meshes/Puzzlebot_Caster_Wheel.stl"/>
       </geometry>
       <material name="grey">
@@ -109,6 +112,7 @@
     </visual>
     <collision>
-      <geometry>
-        <sphere radius="0.015"/>
+      <origin xyz="0 0 0.0057" rpy="0 0 0"/>
+      <geometry>
+        <sphere radius="0.0115"/>
       </geometry>
     </collision>
@@ -172,5 +176,5 @@
     <parent link="base_link"/>
     <child link="wheel_right_link"/>
-    <origin xyz="0.052 -0.095 -0.0025" rpy="0.0 0.0 0.0"/>
+    <origin xyz="0.052 -0.095 0.0" rpy="0.0 0.0 0.0"/>
     <axis xyz="0 1 0"/>
   </joint>
@@ -179,12 +183,14 @@
     <parent link="base_link"/>
     <child link="wheel_left_link"/>
-    <origin xyz="0.052 0.095 -0.0025" rpy="0.0 0.0 0.0"/>
+    <origin xyz="0.052 0.095 0.0" rpy="0.0 0.0 0.0"/>
     <axis xyz="0 1 0"/>
   </joint>
   <!-- base_link -> caster_link -->
+  <!-- z=-0.0442: places ball bottom (mesh z_min=-0.0058) at world z=0 when
+       base_link is at z=0.05 and drive wheels (r=0.05) rest on the ground. -->
   <joint name="caster_joint" type="fixed">
     <parent link="base_link"/>
     <child link="caster_link"/>
-    <origin xyz="-0.095 0.0 -0.03" rpy="0.0 0.0 0.0"/>
+    <origin xyz="-0.095 0.0 -0.0432" rpy="0.0 0.0 0.0"/>
   </joint>
   <!-- base_link -> lidar_link -->

File: src/description/urdf/puzzlebot_gazebo.xacro (robot description, xacro)
@@ -33,15 +33,12 @@
     <xacro:if value="$(arg is_ignition)">
       <plugin filename="ign_ros2_control-system" name="ign_ros2_control::IgnitionROS2ControlPlugin">
-        <parameters>$(find puzzlebot_controller)/config/puzzlebot_controllers.yaml</parameters>
+        <parameters>$(find controller)/config/puzzlebot_controllers.yaml</parameters>
       </plugin>
-      <plugin filename="ignition-gazebo-imu-system" name="ignition::gazebo::systems::Imu">
-      </plugin>
-      <plugin filename="ignition-gazebo-sensors-system" name="ignition::gazebo::systems::Sensors">
-        <render_engine>ogre2</render_engine>
-      </plugin>
+      <!-- IMU and Sensors (ogre2) plugins omitted: gpu rendering unavailable
+           in this headless environment. Re-enable when running on the Jetson. -->
     </xacro:if>
     <xacro:unless value="$(arg is_ignition)">
       <plugin filename="gz_ros2_control-system" name="gz_ros2_control::GazeboSimROS2ControlPlugin">
-        <parameters>$(find puzzlebot_controller)/config/puzzlebot_controllers.yaml</parameters>
+        <parameters>$(find controller)/config/puzzlebot_controllers.yaml</parameters>
       </plugin>
       <plugin filename="gz-sim-imu-system" name="gz::sim::systems::Imu">
@@ -103,5 +100,5 @@
     </sensor>
   </gazebo>
-  <!-- 2D Lidar sensor -->
+  <!-- 2D Lidar sensor (gpu_lidar uses render engine for raycasting in Ignition) -->
   <gazebo reference="lidar_link">
     <sensor name="lidar" type="gpu_lidar">
@@ -122,5 +119,5 @@
         <range>
           <min>0.12</min>
-          <max>12.0</max>
+          <max>20.0</max>
           <resolution>0.02</resolution>
         </range>
