Commit message: Integra mapeo real y description completo desde testing
- Agrega real_odom.py y real.launch.py para odometría en hardware real
- Agrega mapping_real.launch.py y actualiza mapping.launch.py para SLAM real
- Actualiza slam_node.py con mejoras de testing
- Reorganiza meshes en subdirectorios: lifter/, other/, rollers/
- Agrega meshes nuevos: UpperCase, camera, camera_holder, mast_inner, rollers
- Actualiza URDFs: lifter, puzzlebot_with_lifter, puzzlebot_gazebo, puzzlebot_mcr2, ros2_control
- Agrega mundo new_warehouse.world, actualiza obstacles.world
- Actualiza warehouse_rack model.config y model.sdf

Co-Authored-By: Claude Sonnet 4.6 <noreply@anthropic.com>

File: src/description/urdf/puzzlebot_with_lifter.urdf.xacro (robot description, xacro)
@@ -5,7 +5,7 @@
   <xacro:arg name="is_sim" default="true"/>
   <!-- Include Gazebo plugins -->
-  <xacro:include filename="$(find puzzlebot_description)/urdf/puzzlebot_gazebo.xacro" />
+  <xacro:include filename="$(find description)/urdf/puzzlebot_gazebo.xacro" />
   <!-- Include ros2_control -->
-  <xacro:include filename="$(find puzzlebot_description)/urdf/puzzlebot_ros2_control.xacro" />
+  <xacro:include filename="$(find description)/urdf/puzzlebot_ros2_control.xacro" />
   <!-- ==================== PROPERTIES ==================== -->
   <xacro:property name="wheel_radius"    value="0.05"/>
@@ -47,5 +47,5 @@
     <visual>
       <geometry>
-        <mesh filename="package://puzzlebot_description/meshes/Puzzlebot_Jetson_Lidar_Edition_Base.stl"/>
+        <mesh filename="package://description/meshes/Puzzlebot_Jetson_Lidar_Edition_Base.stl"/>
       </geometry>
       <material name="dark_grey">
@@ -64,5 +64,5 @@
       <origin xyz="0 0 0" rpy="-1.5708 0 0"/>
       <geometry>
-        <mesh filename="package://puzzlebot_description/meshes/Puzzlebot_Wheel.stl"/>
+        <mesh filename="package://description/meshes/Puzzlebot_Wheel.stl"/>
       </geometry>
       <material name="grey">
@@ -82,5 +82,5 @@
       <origin xyz="0 0 0" rpy="1.5708 0 0"/>
       <geometry>
-        <mesh filename="package://puzzlebot_description/meshes/Puzzlebot_Wheel.stl"/>
+        <mesh filename="package://description/meshes/Puzzlebot_Wheel.stl"/>
       </geometry>
       <material name="grey">
@@ -98,6 +98,7 @@
     <xacro:sphere_inertia m="${caster_mass}" r="0.015"/>
     <visual>
-      <geometry>
-        <mesh filename="package://puzzlebot_description/meshes/Puzzlebot_Caster_Wheel.stl"/>
+      <origin xyz="0 0 -0.015" rpy="0 0 0"/>
+      <geometry>
+        <mesh filename="package://description/meshes/Puzzlebot_Caster_Wheel.stl"/>
       </geometry>
       <material name="grey">
@@ -160,7 +161,7 @@
   <link name="lifter_base_link">
     <visual>
-      <origin xyz="-0.1125 0.0112 -0.1125" rpy="1.5708 0 0"/>
-      <geometry>
-        <mesh filename="package://puzzlebot_description/meshes/4-mast-1.stl"
+      <origin xyz="-0.1125 -0.0112 0.1125" rpy="1.5708 3.14159 3.14159"/>
+      <geometry>
+        <mesh filename="package://description/meshes/lifter/outer_mast.stl"
               scale="${s} ${s} ${s}"/>
       </geometry>
@@ -182,11 +183,11 @@
     </inertial>
   </link>
-  <!-- Inner mast (7-mast-2.stl)
-       Physical size in world frame: 49 × 11.6 × 155.5 mm -->
+  <!-- Inner mast (Frantic Albar-Hillar (9).stl)
+       Physical size in world frame: 49 × 11.6 × 171 mm -->
   <link name="mast_inner_link">
     <visual>
-      <origin xyz="-0.1125 0.0058 -0.1125" rpy="1.5708 0 0"/>
-      <geometry>
-        <mesh filename="package://puzzlebot_description/meshes/7-mast-2.stl"
+      <origin xyz="-0.0655 0.0058 -0.0050" rpy="1.5708 0 0"/>
+      <geometry>
+        <mesh filename="package://description/meshes/lifter/mast_inner.stl"
               scale="${s} ${s} ${s}"/>
       </geometry>
@@ -198,5 +199,5 @@
       <origin xyz="0 0 0" rpy="0 0 0"/>
       <geometry>
-        <box size="0.049 0.0116 0.1555"/>
+        <box size="0.049 0.0116 0.171"/>
       </geometry>
     </collision>
@@ -214,5 +215,5 @@
       <origin xyz="-0.1125 -0.11343 -0.02793" rpy="0 0 0"/>
       <geometry>
-        <mesh filename="package://puzzlebot_description/meshes/8-carriage.stl"
+        <mesh filename="package://description/meshes/lifter/carriage.stl"
               scale="${s} ${s} ${s}"/>
       </geometry>
@@ -232,4 +233,52 @@
       <inertia ixx="0.0000207" ixy="0" ixz="0"
                iyy="0.0000159" iyz="0" izz="0.0000262"/>
+    </inertial>
+  </link>
+  <!-- Camera pan holder (camera_holder.stl) — rotates on top of inner mast -->
+  <link name="cam_holder_link">
+    <visual>
+      <origin xyz="0.0285 -0.0055 0.0715" rpy="-1.5708 0 0"/>
+      <geometry>
+        <mesh filename="package://description/meshes/lifter/camera_holder.stl"
+              scale="${s} ${s} ${s}"/>
+      </geometry>
+      <material name="light_grey">
+        <color rgba="0.80 0.80 0.75 1.0"/>
+      </material>
+    </visual>
+    <collision>
+      <origin xyz="0 0 0.01125" rpy="0 0 0"/>
+      <geometry>
+        <box size="0.041 0.009 0.0225"/>
+      </geometry>
+    </collision>
+    <inertial>
+      <origin xyz="0 0 0.01125" rpy="0 0 0"/>
+      <mass value="0.01"/>
+      <inertia ixx="1e-6" ixy="0" ixz="0" iyy="1e-6" iyz="0" izz="1e-6"/>
+    </inertial>
+  </link>
+  <!-- Mast camera (camera.stl) — fixed to the pan holder -->
+  <link name="mast_camera_link">
+    <visual>
+      <origin xyz="-0.0005 0.0290 0.0005" rpy="-1.5708 0 3.14159"/>
+      <geometry>
+        <mesh filename="package://description/meshes/lifter/camera.stl"
+              scale="${s} ${s} ${s}"/>
+      </geometry>
+      <material name="black">
+        <color rgba="0.1 0.1 0.1 1.0"/>
+      </material>
+    </visual>
+    <collision>
+      <origin xyz="0 0 0" rpy="0 0 0"/>
+      <geometry>
+        <box size="0.041 0.041 0.014"/>
+      </geometry>
+    </collision>
+    <inertial>
+      <origin xyz="0 0 0" rpy="0 0 0"/>
+      <mass value="0.01"/>
+      <inertia ixx="1e-6" ixy="0" ixz="0" iyy="1e-6" iyz="0" izz="1e-6"/>
     </inertial>
   </link>
@@ -255,10 +304,10 @@
     <parent link="base_link"/>
     <child  link="caster_link"/>
-    <origin xyz="-0.095 0.0 -0.03" rpy="0.0 0.0 0.0"/>
+    <origin xyz="-0.095 0 -0.0307" rpy="0 0 0"/>
   </joint>
   <joint name="lidar_joint" type="fixed">
     <parent link="base_link"/>
     <child  link="lidar_link"/>
-    <origin xyz="0.0 0.0 0.08" rpy="0.0 0.0 0.0"/>
+    <origin xyz="0.04 0.0 0.12" rpy="0.0 0.0 0.0"/>
   </joint>
   <joint name="camera_joint" type="fixed">
@@ -301,4 +350,17 @@
     <dynamics damping="10.0" friction="2.0"/>
   </joint>
+  <!-- Pan holder: revolute around X at top of inner mast -->
+  <joint name="cam_holder_joint" type="fixed">
+    <parent link="mast_inner_link"/>
+    <child  link="cam_holder_link"/>
+    <origin xyz="0 0 0.105" rpy="0.7854 0 0"/>
+  </joint>
+  <!-- Camera: fixed to the pan holder, sits on top of bracket
+       z=0.030: bracket top (0.0225) + half camera height (0.007) = 0.0295 ≈ 0.030m -->
+  <joint name="mast_camera_joint" type="fixed">
+    <parent link="cam_holder_link"/>
+    <child  link="mast_camera_link"/>
+    <origin xyz="0 0 0.033" rpy="0 0 0"/>
+  </joint>
   <!-- ==================== MATERIALS ==================== -->
   <material name="dark_grey">
