Commit message: Fix mapping_real: real_odom crash, URDF mesh roto, TF conflict, RViz crash
- real_odom: reemplaza tf_transformations (np.float incompatible con NumPy 1.20+)
  con función _quat_from_yaw usando math puro
- puzzlebot_mcr2.urdf.xacro: apunta a Puzzlebot_Jetson_Lidar_Edition_Base.stl
  (MCR2_puzzlebot_jetson_lidar_base.stl fue eliminado al reorganizar meshes)
- mapping_real.launch.py: elimina static TF odom->base_footprint que conflictúa
  con el TF dinámico de real_odom; actualiza argumentos deprecated de
  static_transform_publisher a nuevo estilo --frame-id/--child-frame-id
- slam.rviz: elimina panel Image /video_source/raw que causaba crash inmediato de RViz

Co-Authored-By: Claude Sonnet 4.6 <noreply@anthropic.com>

File: src/description/urdf/puzzlebot_mcr2.urdf.xacro (robot description, xacro)
@@ -51,5 +51,5 @@
       <origin xyz="0.050 0 0.0965" rpy="1.5708 0 3.1416"/>
       <geometry>
-        <mesh filename="package://description/meshes/MCR2_puzzlebot_jetson_lidar_base.stl"/>
+        <mesh filename="package://description/meshes/Puzzlebot_Jetson_Lidar_Edition_Base.stl"/>
       </geometry>
       <material name="dark_grey">
