Commit message: Testing Real and Sim launch files

File: src/description/urdf/puzzlebot_mcr2.urdf.xacro (robot description, xacro)
@@ -5,7 +5,7 @@
   <xacro:arg name="is_sim" default="true"/>
   <!-- Include Gazebo plugins -->
-  <xacro:include filename="$(find puzzlebot_description)/urdf/puzzlebot_gazebo.xacro" />
+  <xacro:include filename="$(find description)/urdf/puzzlebot_gazebo.xacro" />
   <!-- Include ros2_control -->
-  <xacro:include filename="$(find puzzlebot_description)/urdf/puzzlebot_ros2_control.xacro" />
+  <xacro:include filename="$(find description)/urdf/puzzlebot_ros2_control.xacro" />
   <!-- ==================== PROPERTIES ==================== -->
   <xacro:property name="wheel_radius" value="0.05"/>
@@ -51,5 +51,5 @@
       <origin xyz="0.050 0 0.0965" rpy="1.5708 0 3.1416"/>
       <geometry>
-        <mesh filename="package://puzzlebot_description/meshes/MCR2_puzzlebot_jetson_lidar_base.stl"/>
+        <mesh filename="package://description/meshes/MCR2_puzzlebot_jetson_lidar_base.stl"/>
       </geometry>
       <material name="dark_grey">
@@ -69,5 +69,5 @@
       <origin xyz="0.055 -0.0048 0" rpy="1.57 0 0"/>
       <geometry>
-        <mesh filename="package://puzzlebot_description/meshes/MCR2_wheel.stl"/>
+        <mesh filename="package://description/meshes/MCR2_wheel.stl"/>
       </geometry>
       <material name="grey">
@@ -88,5 +88,5 @@
       <origin xyz="0.055 0.0048 0" rpy="-1.57 0 0"/>
       <geometry>
-        <mesh filename="package://puzzlebot_description/meshes/MCR2_wheel.stl"/>
+        <mesh filename="package://description/meshes/MCR2_wheel.stl"/>
       </geometry>
       <material name="grey">
@@ -107,5 +107,5 @@
       <origin xyz="0 0 -0.015" rpy="0 0 0"/>
       <geometry>
-        <mesh filename="package://puzzlebot_description/meshes/MCR2_caster_wheel.stl"/>
+        <mesh filename="package://description/meshes/MCR2_caster_wheel.stl"/>
       </geometry>
       <material name="grey">

Commit message: Update real mapping

File: src/description/urdf/puzzlebot_mcr2.urdf.xacro (robot description, xacro)
@@ -51,5 +51,5 @@
       <origin xyz="0.050 0 0.0965" rpy="1.5708 0 3.1416"/>
       <geometry>
-        <mesh filename="package://description/meshes/Puzzlebot_Jetson_Lidar_Edition_Base.stl"/>
+        <mesh filename="package://description/meshes/MCR2_puzzlebot_jetson_lidar_base.stl"/>
       </geometry>
       <material name="dark_grey">

File: src/description/urdf/puzzlebot_with_lifter.urdf.xacro (robot description, xacro)
@@ -4,4 +4,7 @@
   <xacro:arg name="is_ignition" default="true"/>
   <xacro:arg name="is_sim" default="true"/>
+  <!-- LiDAR is mounted rear-facing on the real robot (cable toward back).
+       Rotate 180° in real mode so the scan aligns with +X forward. -->
+  <xacro:property name="lidar_yaw" value="${0.0 if '$(arg is_sim)' == 'true' else 3.141592653589793}"/>
   <!-- Include Gazebo plugins -->
   <xacro:include filename="$(find description)/urdf/puzzlebot_gazebo.xacro" />
@@ -14,8 +17,4 @@
   <xacro:property name="wheel_mass" value="0.1"/>
   <xacro:property name="caster_mass" value="0.01"/>
-  <!-- Real RPLidar A1 is mounted 180° rotated (motor/cable at front).
-       Simulation emits rays from +X so no correction is needed there. -->
-  <xacro:property name="lidar_yaw"
-    value="${0.0 if '$(arg is_sim)' == 'true' else 3.141592653589793}"/>
   <!-- mm → m for lifter STL meshes -->
   <xacro:property name="s" value="0.001"/>
