Commit message: Fix robot model: usa puzzlebot_with_lifter URDF y corrige paths de lifter
- mapping_real.launch.py: cambia URDF de puzzlebot_mcr2 a puzzlebot_with_lifter
  para que RViz muestre el robot completo con lifter, cámara y LiDAR como cilindro
- lifter.urdf.xacro: corrige 5 paths de package://puzzlebot_description/ a
  package://description/ (nombre de paquete renombrado)

Co-Authored-By: Claude Sonnet 4.6 <noreply@anthropic.com>

File: src/description/urdf/lifter.urdf.xacro (robot description, xacro)
@@ -21,5 +21,5 @@
       <origin xyz="-0.1125 -0.0112 0.1125" rpy="1.5708 3.14159 3.14159"/>
       <geometry>
-        <mesh filename="package://puzzlebot_description/meshes/lifter/outer_mast.stl"
+        <mesh filename="package://description/meshes/lifter/outer_mast.stl"
               scale="${s} ${s} ${s}"/>
       </geometry>
@@ -41,5 +41,5 @@
       <origin xyz="-0.0655 0.0058 -0.0050" rpy="1.5708 0 0"/>
       <geometry>
-        <mesh filename="package://puzzlebot_description/meshes/lifter/mast_inner.stl"
+        <mesh filename="package://description/meshes/lifter/mast_inner.stl"
               scale="${s} ${s} ${s}"/>
       </geometry>
@@ -62,5 +62,5 @@
       <origin xyz="-0.1125 -0.11343 -0.02793" rpy="0 0 0"/>
       <geometry>
-        <mesh filename="package://puzzlebot_description/meshes/lifter/carriage.stl"
+        <mesh filename="package://description/meshes/lifter/carriage.stl"
               scale="${s} ${s} ${s}"/>
       </geometry>
@@ -82,5 +82,5 @@
       <origin xyz="0.0285 -0.0055 0.0715" rpy="-1.5708 0 0"/>
       <geometry>
-        <mesh filename="package://puzzlebot_description/meshes/lifter/camera_holder.stl"
+        <mesh filename="package://description/meshes/lifter/camera_holder.stl"
               scale="${s} ${s} ${s}"/>
       </geometry>
@@ -99,5 +99,5 @@
       <origin xyz="-0.0005 0.0290 0.0005" rpy="-1.5708 0 3.14159"/>
       <geometry>
-        <mesh filename="package://puzzlebot_description/meshes/lifter/camera.stl"
+        <mesh filename="package://description/meshes/lifter/camera.stl"
               scale="${s} ${s} ${s}"/>
       </geometry>
